File: hardware/pcb/gdep133c02-driver/gdep133c02-driver.kicad_pcb (KiCad board)
At the start: 4 copper layers, 100 x 80 mm, 158 parts, among them J1 3V3 BENCH ONLY, J2 HOST 3V3 LOGIC, Q1 DMN3065LW-7, Q10 2N7002-7-F, Q3 MMBT3906-7-F, Q4 DMN3065LW-7, Q6 MMBT3904-7-F, Q7 PJA3433_R1_00001, Q8 DMP3068L-7, Q9 2N7002-7-F, U1 0.2 ohm, U2 0.2 ohm, U3 0.2 ohm, U4 TCN75AVOA713, U5 TPS22913BYZVT, U6 SN74LVC244APWR, U7 SN74LVC244APWR

Commit message: save
Parts:
- removed C34, C35: 100nF/50V, Driver:Capacitor_SMD__C_0603_1608Metric
- removed L4: BLM18PG221SH1D, Driver:Inductor_SMD__L_0603_1608Metric
- removed L5: CBG160808U000T, Driver:Inductor_SMD__L_0603_1608Metric
- removed Q10, Q9: 2N7002-7-F, Driver:Package_TO_SOT_SMD__SOT-23
- removed R14, R15, R16, R23, R24, R25, R29, R33, R34, R4, R5, R6, R9: 0 ohm, Driver:Resistor_SMD__R_0603_1608Metric
- removed R22, R37, R38: 10k ohm, Driver:Resistor_SMD__R_0603_1608Metric
- removed R26, R27, R28, R31, R32: 0 ohm, Driver:Resistor_SMD__R_1206_3216Metric
- removed U6, U7: SN74LVC244APWR, Driver:Package_SO__TSSOP-20_4.4x6.5mm_P0.65mm
- added C36: 1nF/50V C0G, Driver:Capacitor_SMD__C_0805_2012Metric, F.Cu at (87.0, 125.0)
- J2: value HOST 3V3 LOGIC -> HOST DIRECT 3V3
- TP2: value VIN -> EPD_3V3
- TP3: value AVDD -> EPD_3V3
- U5: value TPS22913BYZVT -> TPS22917DBVR; footprint Driver:Package_CSP__WLCSP-4_0.89x0.89mm_Layout2x2_P0.5mm -> Driver:Package_TO_SOT_SMD__SOT-23-6
Connections:
- C12 pad 1: AVDD -> EPD_3V3
- C14 pad 1: AVDD -> EPD_3V3
- C16 pad 1: VGH_RAW -> VGH
- C19 pad 1: AVDD -> EPD_3V3
- C28 pad 1: EPD_VDD -> BENCH_3V3
- C29 pad 1: VIN -> EPD_3V3
- C30 pad 1: VIN -> EPD_3V3
- C31 pad 1: AVDD_CAP -> EPD_3V3
- C32 pad 1: AVDD_CAP -> EPD_3V3
- D2 pad 2: VDDN_RAW -> VDDN
- D3 pad 2: VGH_RAW -> VGH
- FPC1 pad 10: VDD -> EPD_3V3
- FPC1 pad 19: VDDIO -> EPD_3V3
- FPC1 pad 22: BS0 -> EPD_3V3
- FPC1 pad 23: BS1 -> EPD_3V3
- FPC1 pad 41: VNCP_3P5V -> VBB_3P5V
- FPC1 pad 9: AVDD -> EPD_3V3
- J2 pad 13: HOST_BUSY_N -> BUSY_N
- J2 pad 16: HOST_3V3 -> unconnected-(J2-NC-Pad16)
- J2 pad 5: HOST_MISO -> SI1
- L1 pad 1: AVDD -> EPD_3V3
- Q7 pad 1: GATE_VCOM -> GDRC
- Q7 pad 2: SENSE_VCOM -> RESEC
- Q8 pad 1: GATE_N -> GDRN
- Q8 pad 2: SENSE_N -> RESEN
- R1 pad 2: VDDIO -> EPD_3V3
- R13 pad 1: AVDD -> EPD_3V3
- R13 pad 2: GATE_VCOM -> GDRC
- R3 pad 1: AVDD -> EPD_3V3
- R3 pad 2: GATE_N -> GDRN
- R30 pad 1: SW_ON -> EPD_PWR_EN
- R39 pad 1: BUF_SCLK -> HOST_SCLK
- R40 pad 1: BUF_MOSI -> HOST_MOSI
- R41 pad 1: BUF_CS_M_N -> HOST_CS_M_N
- R42 pad 1: BUF_CS_S_N -> HOST_CS_S_N
- R43 pad 1: BUF_RES_N -> HOST_RES_N
- R46 pad 2: VDDIO -> EPD_3V3
- R47 pad 2: VDDIO -> EPD_3V3
- R8 pad 2: VGH_RAW -> VGH
- TP10 pad 1: VNCP_3P5V -> VBB_3P5V
- TP2 pad 1: VIN -> EPD_3V3
- TP3 pad 1: AVDD -> EPD_3V3
- U2 pad 1: AVDD -> EPD_3V3
- U2 pad 2: SENSE_N -> RESEN
- U3 pad 1: AVDD -> EPD_3V3
- U3 pad 2: SENSE_VCOM -> RESEC
- U4 pad 3: ALERT_N -> unconnected-(U4-ALERT_N-Pad3)
Routing:
- net EPD_3V3: track 163.3 -> 680.0 mm, vias 4 -> 18
- net AVDD: track 172.3 -> 0.00 mm, vias 2 -> 0
- net VDDIO: track 114.8 -> 0.00 mm, vias 3 -> 0
- net VDD: track 85.2 -> 0.00 mm, vias 4 -> 0
- net VBB_3P5V: track 77.9 -> 154.4 mm, vias 2 -> 6
- net VNCP_3P5V: track 74.9 -> 0.00 mm, vias 4 -> 0
- net VIN: track 61.1 -> 0.00 mm
- net BUF_SCLK: track 35.2 -> 0.00 mm, vias 2 -> 0
- net BUF_MOSI: track 30.0 -> 0.00 mm, vias 2 -> 0
- net AVDD_CAP: track 27.8 -> 0.00 mm
- net BENCH_3V3: track 11.5 -> 38.4 mm, vias 0 -> 4
- net ALERT_N: track 25.8 -> 0.00 mm
- net BUSY_N: track 94.9 -> 120.5 mm, vias 3 -> 4
- net BUF_CS_M_N: track 25.1 -> 0.00 mm, vias 4 -> 0
- net BS1: track 22.2 -> 0.00 mm, vias 2 -> 0
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
Commit message: save
Parts:
- added R49: 0 ohm, Driver:Resistor_SMD__R_0805_2012Metric, F.Cu at (108.9, 93.7)
- added TP25: GDRC, Driver:TestPoint__TestPoint_Pad_D1.5mm, F.Cu at (104.5, 94.0)
- added TP26: Q7_GATE, Driver:TestPoint__TestPoint_Pad_D1.5mm, F.Cu at (106.0, 98.5)
Connections:
- Q7 pad 1: GDRC -> Q7_GATE
- R13 pad 2: GDRC -> Q7_GATE
Routing:
- net Q7_GATE: track 0.00 -> 12.4 mm, vias 0 -> 2
- net GDRC: track 63.0 -> 56.8 mm, vias 3 -> 4
