File: hardware/pcb/gdep133c02-driver/interface.kicad_sch (KiCad schematic)
At the start: 43 parts, among them J2 HOST 3V3 LOGIC, Q10 2N7002-7-F, Q9 2N7002-7-F, U6 SN74LVC244APWR, U7 SN74LVC244APWR

Commit message: save
Other:
- note added: "1 Host connector - 3.3V logic / common ground"
- note added: "2 Host to panel - buffered SPI / default levels"
- note added: "3 Panel to host - BUSY / MISO buffer"
- note added: "4 Power test points"
- note added: "5 Control test points / common ground pads"
- note added: "Dots join wires; crossings without dots do not connect. Global labels retain existing PCB net names."
- note added: "EPD_PWR_EN high: Q9 pulls both OE inputs low."
- note added: "J2.16 powers host-side logic only."
- note added: "TP1-TP24 are copper pads; DNP crosses mean no assembled component, not an unconnected pin."
- note added: "Unused inputs grounded; unused outputs marked NC."
- title: Host isolation and test points -> Interface - wired functional circuits
- moved on the sheet: J2

Commit message: save
Parts:
- removed C34: 100nF/50V, Driver:Capacitor_SMD__C_0603_1608Metric, symbol Driver:P_C34
- removed C35: 100nF/50V, Driver:Capacitor_SMD__C_0603_1608Metric, symbol Driver:P_C35
- removed Q10: 2N7002-7-F, Driver:Package_TO_SOT_SMD__SOT-23, symbol Driver:P_Q10
- removed Q9: 2N7002-7-F, Driver:Package_TO_SOT_SMD__SOT-23, symbol Driver:P_Q9
- removed R37: 10k ohm, Driver:Resistor_SMD__R_0603_1608Metric, symbol Driver:P_R37
- removed R38: 10k ohm, Driver:Resistor_SMD__R_0603_1608Metric, symbol Driver:P_R38
- removed U6: SN74LVC244APWR, Driver:Package_SO__TSSOP-20_4.4x6.5mm_P0.65mm, symbol Driver:P_U6
- removed U7: SN74LVC244APWR, Driver:Package_SO__TSSOP-20_4.4x6.5mm_P0.65mm, symbol Driver:P_U7
- J2: value HOST 3V3 LOGIC -> HOST DIRECT 3V3
- TP2: value VIN -> EPD_3V3
- TP3: value AVDD -> EPD_3V3
Connections:
- net AVDD is gone; now on net EPD_3V3: TP3.1
- net BUF_CS_M_N is gone; now on net HOST_CS_M_N: R41.1
- net BUF_CS_S_N is gone; now on net HOST_CS_S_N: R42.1
- net BUF_MOSI is gone; now on net HOST_MOSI: R40.1
- net BUF_RES_N is gone; now on net HOST_RES_N: R43.1
- net BUF_SCLK is gone; now on net HOST_SCLK: R39.1
- net HOST_BUSY_N is gone; now on net BUSY_N: J2.13 (BUSY_N)
- net HOST_MISO is gone; now on net SI1: J2.5 (MISO)
- net VDDIO is gone; now on net EPD_3V3: R46.2, R47.2
- net VIN is gone; now on net EPD_3V3: TP2.1
- net VNCP_3P5V is gone; now on net VBB_3P5V: TP10.1
- net HOST_3V3: no longer names the net of J2.16 (NC)
- no-connect marks 9 -> 1
Other:
- note added: "Direct 3.3V host interface - NO power-off signal isolation"
- note added: "Host first ON / last OFF. Screen OFF: no GPIO HIGH, no pull-ups."
- note added: "J2.16 unused. No live plugging. Short cable <= 10cm."
- note added: "Test pads: copper only, no parts to buy or solder"
- note removed: "1 Host connector - 3.3V logic / common ground"
- note removed: "2 Host to panel - buffered SPI / default levels"
- note removed: "3 Panel to host - BUSY / MISO buffer"
- note removed: "4 Power test points"
- note removed: "5 Control test points / common ground pads"
- note removed: "Dots join wires; crossings without dots do not connect. Global labels retain existing PCB net names."
- note removed: "EPD_PWR_EN high: Q9 pulls both OE inputs low."
- note removed: "J2.16 powers host-side logic only."
- note removed: "TP1-TP24 are copper pads; DNP crosses mean no assembled component, not an unconnected pin."
- note removed: "Unused inputs grounded; unused outputs marked NC."
- moved on the sheet: R39, R40, R41, R42, R43, R44, R45, R46, R47, R48, TP1, TP10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

Commit message: save
Parts:
- J2: BOM Comments (none) -> 首韩2×8直插排针；原厂图20.32×5.0mm、2.54mm双排、0.64mm方针、3A；孔径1.05mm。; LCSC (none) -> C55629829; MPN TSW-108-07-G-D -> SH-PZ254V-2x8P; Manufacturer Samtec -> SHOU HAN
- R39, R40, R41, R42, R43: footprint Driver:Resistor_SMD__R_0603_1608Metric -> Driver:R_0805_HandSolder; BOM Comments (none) -> 同阻值±1%常用0805；手焊加长焊盘。; LCSC (none) -> C17634; MPN RC0603FR-0733RL -> 0805W8F330JT5E; Manufacturer Yageo -> UNI-ROYAL
- R44, R45, R46, R47, R48: footprint Driver:Resistor_SMD__R_0603_1608Metric -> Driver:R_0805_HandSolder; BOM Comments (none) -> 同阻值±1%常用0805；手焊加长焊盘。; LCSC (none) -> C149504; MPN RC0603FR-07100KL -> 0805W8F1003T5E; Manufacturer Yageo -> UNI-ROYAL
- TP1, TP10, TP11, TP12, TP13, TP14, TP15, TP16, TP17, TP18, TP19, TP2, TP20, TP21, TP22, TP23, TP24, TP3, TP4, TP5, TP6, TP7, TP8, TP9: BOM Comments (none) -> 保留原型号/封装；本轮逐项复核，关键动态参数未有充分替代证据。
