File: hardware/pcb/gdep133c02-driver/panel.kicad_sch (KiCad schematic)
At the start: 41 parts, among them U4 TCN75AVOA713

Commit message: save
Other:
- note added: "1 Screen connector - pin numbers retained; functional pin layout"
- note added: "2 SPI mode / signal defaults"
- note added: "3 Panel-controlled temperature sensor"
- note added: "4 Source outputs / input straps / capacitor banks"
- note added: "Dots join wires; crossings without dots do not connect. Global labels are cross-sheet interfaces."
- note added: "Nominal 33.3uF; effective capacitance pending."
- note added: "R23 DNP: alert output is not strapped to ground."
- note added: "Symbol grouping does not represent physical FPC pin positions."
- title: Panel and temperature -> Panel - wired functional circuits
- moved on the sheet: U4

Commit message: save
Parts:
- removed R22: 10k ohm, Driver:Resistor_SMD__R_0603_1608Metric, symbol Driver:P_R22
- removed R23: 0 ohm, Driver:Resistor_SMD__R_0603_1608Metric, symbol Driver:P_R23
- removed R24: 0 ohm, Driver:Resistor_SMD__R_0603_1608Metric, symbol Driver:P_R24
- removed R25: 0 ohm, Driver:Resistor_SMD__R_0603_1608Metric, symbol Driver:P_R25
Connections:
- net AVDD is gone; now on net EPD_3V3: FPC1.9 (AVDD)
- net BS0 is gone; now on net EPD_3V3: FPC1.22 (BS0)
- net BS1 is gone; now on net EPD_3V3: FPC1.23 (BS1)
- net VDD is gone; now on net EPD_3V3: FPC1.10 (VDD)
- net VDDIO is gone; now on net EPD_3V3: FPC1.19 (VDDIO), R1.2
- net VNCP_3P5V is gone; now on net VBB_3P5V: FPC1.41 (VNCP_3P5V)
- net ALERT_N: no longer names the net of U4.3 (ALERT_N)
- no-connect marks 4 -> 5

Commit message: save
Parts:
- C1, C103, C104, C106, C107, C109, C110, C112, C113, C115, C116, C118, C119, C2, C3, C4, C5, C6, C7: BOM Comments (none) -> 保留原型号/封装；本轮逐项复核，关键动态参数未有充分替代证据。; LCSC (none) -> C77102
- C10, C11, C9: BOM Comments (none) -> 保留Murata470nF/50V：三星候选未取得工作偏压有效容量及纹波对照。
- C105, C108, C111, C114, C117, C120: BOM Comments (none) -> 保留原型号/封装；本轮逐项复核，关键动态参数未有充分替代证据。
- C27: footprint Driver:Capacitor_SMD__C_0603_1608Metric -> Driver:C_0805_HandSolder; BOM Comments (none) -> 100nF/50V X7R±10%；0603增大为0805。; LCSC (none) -> C1711; MPN GRM188R71H104KA93D -> CL21B104KBCNNNC; Manufacturer Murata -> Samsung
- C8: BOM Comments (none) -> 保留原型号/封装；本轮逐项复核，关键动态参数未有充分替代证据。; LCSC (none) -> C86052
- FPC1: BOM Comments (none) -> 保留原型号/封装；本轮逐项复核，关键动态参数未有充分替代证据。; LCSC (none) -> C2856839
- R1: footprint Driver:Resistor_SMD__R_0603_1608Metric -> Driver:R_0805_HandSolder; BOM Comments (none) -> 同阻值±1%常用0805；手焊加长焊盘。; LCSC (none) -> C17604; MPN RC0603FR-072KL -> 0805W8F2001T5E; Manufacturer Yageo -> UNI-ROYAL
- R20, R21: footprint Driver:Resistor_SMD__R_0603_1608Metric -> Driver:R_0805_HandSolder; BOM Comments (none) -> 同阻值±1%常用0805；手焊加长焊盘。; LCSC (none) -> C17673; MPN RC0603FR-074K7L -> 0805W8F4701T5E; Manufacturer Yageo -> UNI-ROYAL
- R35, R36: footprint Driver:Resistor_SMD__R_0603_1608Metric -> Driver:R_0805_HandSolder; BOM Comments (none) -> 同阻值±1%常用0805；手焊加长焊盘。; LCSC (none) -> C149504; MPN RC0603FR-07100KL -> 0805W8F1003T5E; Manufacturer Yageo -> UNI-ROYAL
- U4: BOM Comments (none) -> 保留原型号/封装；本轮逐项复核，关键动态参数未有充分替代证据。; LCSC (none) -> C144313

Commit message: feat(pcb): release v0.9 with fee-waived resistor selections
Parts:
- C10, C11, C9: LCSC (none) -> C86043
- C105, C108, C111, C114, C117, C120: LCSC (none) -> C397310
Changed lines of the file:
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@@
 		(title "Panel - wired functional circuits")
 		(date "2026-10-09")
-		(rev "0.6-DOMESTIC")
+		(rev "0.9-RESISTORS")
 	)
 	(rectangle
@@
 			)
 		)
-		(property "Datasheet" ""
+		(property "Datasheet" "https://atta.szlcsc.com/upload/public/pdf/source/20200305/C490387_23319AE8C154DEB24C505E6C82A8106A.pdf"
 			(at 30.48 220.98 0)
 			(hide yes)
@@
 			)
 		)
-		(property "LCSC" ""
+		(property "LCSC" "C86043"
 			(at 30.48 220.98 0)
 			(hide yes)
@@
 			)
 		)
-		(property "Datasheet" ""
+		(property "Datasheet" "https://atta.szlcsc.com/upload/public/pdf/source/20200305/C490387_23319AE8C154DEB24C505E6C82A8106A.pdf"
 			(at 55.88 236.22 0)
 			(hide yes)
@@
 			)
 		)
-		(property "LCSC" ""
+		(property "LCSC" "C86043"
 			(at 55.88 236.22 0)
 			(hide yes)
@@
 			)
 		)
-		(property "Datasheet" ""
+		(property "Datasheet" "https://atta.szlcsc.com/upload/public/pdf/source/20200305/C490387_23319AE8C154DEB24C505E6C82A8106A.pdf"
 			(at 223.52 223.52 0)
 			(hide yes)
@@
 			)
 		)
-		(property "LCSC" ""
+		(property "LCSC" "C86043"
 			(at 223.52 223.52 0)
 			(hide yes)
@@
 			)
 		)
-		(property "Datasheet" "https://atta.szlcsc.com/upload/public/pdf/source/20200305/C490387_23319AE8C154DEB24C505E6C82A8106A.pdf"
+		(property "Datasheet" "https://search.murata.co.jp/Ceramy/image/img/A01X/G101/ENG/GRM32ER71H475KA88-01A.pdf"
 			(at 269.24 233.68 0)
 			(hide yes)
@@
 			)
 		)
-		(property "Datasheet" ""
+		(property "Datasheet" "https://atta.szlcsc.com/upload/public/pdf/source/20190712/C397310_8EB97581BD3F98F2177A74ABEE8CEC8B.pdf"
 			(at 375.92 264.16 0)
 			(hide yes)
@@
 			)
 		)
-		(property "LCSC" ""
+		(property "LCSC" "C397310"
 			(at 375.92 264.16 0)
 			(hide yes)
@@
 			)
 		)
-		(property "Datasheet" ""
+		(property "Datasheet" "https://atta.szlcsc.com/upload/public/pdf/source/20190712/C397310_8EB97581BD3F98F2177A74ABEE8CEC8B.pdf"
 			(at 375.92 292.1 0)
 			(hide yes)
@@
 			)
 		)
-		(property "LCSC" ""
+		(property "LCSC" "C397310"
 			(at 375.92 292.1 0)
 			(hide yes)
@@
 			)
 		)
-		(property "Datasheet" ""
+		(property "Datasheet" "https://atta.szlcsc.com/upload/public/pdf/source/20190712/C397310_8EB97581BD3F98F2177A74ABEE8CEC8B.pdf"
 			(at 375.92 320.04 0)
 			(hide yes)
@@
 			)
 		)
-		(property "LCSC" ""
+		(property "LCSC" "C397310"
 			(at 375.92 320.04 0)
 			(hide yes)
@@
 			)
 		)
-		(property "Datasheet" ""
+		(property "Datasheet" "https://atta.szlcsc.com/upload/public/pdf/source/20190712/C397310_8EB97581BD3F98F2177A74ABEE8CEC8B.pdf"
 			(at 375.92 347.98 0)
 			(hide yes)
@@
 			)
 		)
-		(property "LCSC" ""
+		(property "LCSC" "C397310"
 			(at 375.92 347.98 0)
 			(hide yes)
@@
 			)
 		)
-		(property "Datasheet" ""
+		(property "Datasheet" "https://atta.szlcsc.com/upload/public/pdf/source/20190712/C397310_8EB97581BD3F98F2177A74ABEE8CEC8B.pdf"
 			(at 375.92 375.92 0)
 			(hide yes)
@@
 			)
 		)
-		(property "LCSC" ""
+		(property "LCSC" "C397310"
 			(at 375.92 375.92 0)
 			(hide yes)
@@
 			)
 		)
-		(property "Datasheet" ""
+		(property "Datasheet" "https://atta.szlcsc.com/upload/public/pdf/source/20190712/C397310_8EB97581BD3F98F2177A74ABEE8CEC8B.pdf"
 			(at 375.92 403.86 0)
 			(hide yes)
@@
 			)
 		)
-		(property "LCSC" ""
+		(property "LCSC" "C397310"
 			(at 375.92 403.86 0)
 			(hide yes)

Commit message: hardware: use Murata C440198 0805 capacitors and release v0.10
Parts:
- C1, C103, C104, C106, C107, C109, C110, C112, C113, C115, C116, C118, C119, C2, C3, C4, C5, C6, C7: value 10uF/50V -> 10uF/50V X5R; footprint Driver:Capacitor_SMD__C_1210_3225Metric -> Driver:C_0805_HandSolder; AssemblyMethod (none) -> SMT; BOM Comments 保留原型号/封装；本轮逐项复核，关键动态参数未有充分替代证据。 -> v0.10 E01指定C440198；X5R/0805；偏压容量与纹波等效未验证；详见E01改版-v0.10.md; ExceptionDecision (none) -> 2026-10-11 user explicitly selected C440198 for E01; protot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; FeeEvidence (none) -> https://item.szlcsc.com/439567.html | SMT基础库; LCSC C77102 -> C440198; LibraryCategory (none) -> 基础库; MPN GRM32ER71H106KA12L -> GRM21BR61H106KE43L; StockQueriedAt (none) -> 2026-10-11T11:28:17.670114+08:00

Commit message: feat(pcb): adopt 17 basic-library groups and release v0.11 prototype
Parts:
- C10, C11, C9: footprint Driver:Capacitor_SMD__C_0805_2012Metric -> Driver:C_0805_HandSolder; AssemblyMethod (none) -> SMT; BOM Comments 保留Murata470nF/50V：三星候选未取得工作偏压有效容量及纹波对照。 -> 2026-10-11 user selected 3+14 groups; E13; PROTOTYPE ONLY -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; ExceptionDecision (none) -> 2026-10-11 user selected 3+14 groups; E13; PROTOTYPE ONLY -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; FeeEvidence (none) -> https://item.szlcsc.com/14623.html | SMT基础库; LCSC C86043 -> C13967; LibraryCategory (none) -> 基础库; MPN GRM21BR71H474KA88L -> CL21B474KBFNNNE; Manufacturer Murata -> Samsung Electro-Mechanics; StockQueriedAt (none) -> 2026-10-11T14:08:21.232417+08:00
- C105, C108, C111, C114, C117, C120: value 3.3uF/50V -> 1uF/50V; footprint Driver:Capacitor_SMD__C_1210_3225Metric -> Driver:C_0805_HandSolder; AssemblyMethod (none) -> SMT; BOM Comments 保留原型号/封装；本轮逐项复核，关键动态参数未有充分替代证据。 -> 2026-10-11 user selected 3+14 groups; E03; PROTOTYPE ONLY -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; ExceptionDecision (none) -> 2026-10-11 user selected 3+14 groups; E03; PROTOTYPE ONLY -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; FeeEvidence (none) -> https://item.szlcsc.com/29074.html | SMT基础库; LCSC C397310 -> C28323; LibraryCategory (none) -> 基础库; MPN GRM32DR71H335KA88L -> CL21B105KBFNNNE; Manufacturer Murata -> Samsung Electro-Mechanics; StockQueriedAt (none) -> 2026-10-11T14:08:23.138241+08:00
- C27: value 100nF/50V -> 100nF/100V; AssemblyMethod (none) -> SMT; BOM Comments 100nF/50V X7R±10%；0603增大为0805。 -> 2026-10-11 user selected 3+14 groups; E21; parametric revie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; ExceptionDecision (none) -> 2026-10-11 user selected 3+14 groups; E21; parametric revie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; FeeEvidence (none) -> https://item.szlcsc.com/28983.html | SMT基础库; LCSC C1711 -> C28233; LibraryCategory (none) -> 基础库; MPN CL21B104KBCNNNC -> CL21B104KCFNNNE; Manufacturer Samsung -> Samsung Electro-Mechanics; StockQueriedAt (none) -> 2026-10-11T14:08:23.039107+08:00
- C8: footprint Driver:Capacitor_SMD__C_1210_3225Metric -> Driver:C_1206_HandSolder; AssemblyMethod (none) -> SMT; BOM Comments 保留原型号/封装；本轮逐项复核，关键动态参数未有充分替代证据。 -> 2026-10-11 user selected 3+14 groups; E05; PROTOTYPE ONLY -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; ExceptionDecision (none) -> 2026-10-11 user selected 3+14 groups; E05; PROTOTYPE ONLY -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; FeeEvidence (none) -> https://item.szlcsc.com/30577.html | SMT基础库; LCSC C86052 -> C29823; LibraryCategory (none) -> 基础库; MPN GRM32ER71H475KA88L -> 1206B475K500NT; Manufacturer Murata -> FH; StockQueriedAt (none) -> 2026-10-11T14:08:16.690356+08:00
