File: hardware/pcb/gdep133c02-driver/power.kicad_sch (KiCad schematic)
At the start: 70 parts, among them J1 3V3 BENCH ONLY, Q1 DMN3065LW-7, Q3 MMBT3906-7-F, Q4 DMN3065LW-7, Q6 MMBT3904-7-F, Q7 PJA3433_R1_00001, Q8 DMP3068L-7, U1 0.2 ohm, U2 0.2 ohm, U3 0.2 ohm, U5 TPS22913BYZVT

Commit message: save
Other:
- note added: "1 3.3V input / load switch / supply distribution"
- note added: "2 Positive source rail (VDDP)"
- note added: "3 Negative source rail (VDDN)"
- note added: "4 VCOM supply branch"
- note added: "5 Positive gate charge pump (VGH)"
- note added: "6 Negative gate charge pump (VGL)"
- note added: "Dots join wires; crossings without dots are not connected. Net labels retain the existing PCB net names."
- title: Power converters -> Power - wired functional circuits
- moved on the sheet: J1, U5

Commit message: save
Parts:
- removed L4: BLM18PG221SH1D, Driver:Inductor_SMD__L_0603_1608Metric, symbol Driver:P_L4
- removed L5: CBG160808U000T, Driver:Inductor_SMD__L_0603_1608Metric, symbol Driver:P_L5
- removed R14: 0 ohm, Driver:Resistor_SMD__R_0603_1608Metric, symbol Driver:P_R14
- removed R15: 0 ohm, Driver:Resistor_SMD__R_0603_1608Metric, symbol Driver:P_R15
- removed R16: 0 ohm, Driver:Resistor_SMD__R_0603_1608Metric, symbol Driver:P_R16
- removed R26: 0 ohm, Driver:Resistor_SMD__R_1206_3216Metric, symbol Driver:P_R26
- removed R27: 0 ohm, Driver:Resistor_SMD__R_1206_3216Metric, symbol Driver:P_R27
- removed R28: 0 ohm, Driver:Resistor_SMD__R_1206_3216Metric, symbol Driver:P_R28
- removed R29: 0 ohm, Driver:Resistor_SMD__R_0603_1608Metric, symbol Driver:P_R29
- removed R31: 0 ohm, Driver:Resistor_SMD__R_1206_3216Metric, symbol Driver:P_R31
- removed R32: 0 ohm, Driver:Resistor_SMD__R_1206_3216Metric, symbol Driver:P_R32
- removed R33: 0 ohm, Driver:Resistor_SMD__R_0603_1608Metric, symbol Driver:P_R33
- removed R34: 0 ohm, Driver:Resistor_SMD__R_0603_1608Metric, symbol Driver:P_R34
- removed R4: 0 ohm, Driver:Resistor_SMD__R_0603_1608Metric, symbol Driver:P_R4
- removed R5: 0 ohm, Driver:Resistor_SMD__R_0603_1608Metric, symbol Driver:P_R5
- removed R6: 0 ohm, Driver:Resistor_SMD__R_0603_1608Metric, symbol Driver:P_R6
- removed R9: 0 ohm, Driver:Resistor_SMD__R_0603_1608Metric, symbol Driver:P_R9
- added C36: 1nF/50V C0G, Driver:Capacitor_SMD__C_0805_2012Metric, symbol Driver:P_C36
- U5: value TPS22913BYZVT -> TPS22917DBVR; footprint Driver:Package_CSP__WLCSP-4_0.89x0.89mm_Layout2x2_P0.5mm -> Driver:Package_TO_SOT_SMD__SOT-23-6; MPN TPS22913BYZVT -> TPS22917DBVR
Connections:
- net AVDD is gone; now on net EPD_3V3: C12.1, C14.1, C19.1, L1.1, R13.1, R3.1, U2.1, U3.1
- net AVDD_CAP is gone; now on net EPD_3V3: C31.1, C32.1
- net EPD_VDD is gone; now on net BENCH_3V3: C28.1
- net GATE_N is gone; now on net GDRN: Q8.1 (G), R3.2
- net GATE_VCOM is gone; now on net GDRC: Q7.1 (G), R13.2
- net SENSE_N is gone; now on net RESEN: Q8.2 (S), U2.2
- net SENSE_VCOM is gone; now on net RESEC: Q7.2 (S), U3.2
- net VDDN_RAW is gone; now on net VDDN: D2.2 (A)
- net VGH_RAW is gone; now on net VGH: C16.1, D3.2 (K), R8.2
- net VIN is gone; now on net EPD_3V3: C29.1, C30.1
- net BENCH_3V3: now also U5.1 (VIN), C36.1
- net EPD_3V3: now also U5.5 (QOD), U5.6 (VOUT)
- net EPD_PWR_EN: now also R30.1, U5.3 (ON)
- net GND: now also U5.2 (GND); no longer U5.B1 (GND)
- removed net SW_IN: U5.A2 (VIN)
- removed net SW_ON: R30.1, U5.B2 (ON)
- removed net SW_OUT: U5.A1 (VOUT)
- new net SW_CT: C36.2, U5.4 (CT)
Other:
- note added: "v0.4: U5 output = EPD_3V3; direct copper feeds to logic and power branches"

Commit message: save
Parts:
- added R49: 0 ohm, Driver:Resistor_SMD__R_0805_2012Metric, symbol Driver:P_R49
- added TP25: GDRC, Driver:TestPoint__TestPoint_Pad_D1.5mm, symbol Driver:P_TP25
- added TP26: Q7_GATE, Driver:TestPoint__TestPoint_Pad_D1.5mm, symbol Driver:P_TP26
Connections:
- net GDRC: now also R49.1, TP25.1; no longer Q7.1 (G), R13.2
- new net Q7_GATE: Q7.1 (G), R13.2, R49.2, TP26.1

Commit message: save
Parts:
- added R50: 200k ohm, Driver:R_0805_HandSolder, symbol Driver:P_R50
- C12, C14, C16, C19, C21, C29, C30: BOM Comments (none) -> 保留原型号/封装；本轮逐项复核，关键动态参数未有充分替代证据。; LCSC (none) -> C86052
- C13, C15, C20: BOM Comments (none) -> 保留原型号/封装；本轮逐项复核，关键动态参数未有充分替代证据。; LCSC (none) -> C77102
- C17, C23, C24: BOM Comments (none) -> 保留原型号/封装；本轮逐项复核，关键动态参数未有充分替代证据。; LCSC (none) -> C86043
- C18: BOM Comments (none) -> 保留原型号/封装；本轮逐项复核，关键动态参数未有充分替代证据。; LCSC (none) -> C86042
- C22, C25: BOM Comments (none) -> 保留原型号/封装；本轮逐项复核，关键动态参数未有充分替代证据。; LCSC (none) -> C77083
- C26: footprint Driver:Capacitor_SMD__C_0603_1608Metric -> Driver:C_0805_HandSolder; BOM Comments (none) -> 47nF/50V X7R±10%；风华0805，保留耐压，动态波形待实测。; LCSC (none) -> C1745; MPN GRM188R71H473KA61D -> 0805B473K500NT; Manufacturer Murata -> FH
- C28, C36, D1, D2, D4, L1, L2, L3, Q7, TP25, TP26, U1, U2, U3: BOM Comments (none) -> 保留原型号/封装；本轮逐项复核，关键动态参数未有充分替代证据。
- C31, C32: BOM Comments (none) -> 保留原型号/封装；本轮逐项复核，关键动态参数未有充分替代证据。; LCSC (none) -> C88154
- C33: footprint Driver:Capacitor_SMD__C_0603_1608Metric -> Driver:C_0805_HandSolder; BOM Comments (none) -> 100nF/50V X7R±10%；0603增大为0805。; LCSC (none) -> C1711; MPN GRM188R71H104KA93D -> CL21B104KBCNNNC; Manufacturer Murata -> Samsung
- D3, D5, D6: BOM Comments (none) -> 保留原型号/封装；本轮逐项复核，关键动态参数未有充分替代证据。; LCSC (none) -> C83574
- J1: BOM Comments (none) -> 国内2.54mm直插排针，3A，孔距及脚序不变。; LCSC (none) -> C42410552; MPN TSW-102-07-G-S -> TJC8-2.54-2A; Manufacturer Samtec -> DLL
- Q1, Q4: footprint Driver:Package_TO_SOT_SMD__SOT-323_SC-70 -> Driver:SOT323_HandSolder; BOM Comments (none) -> 保留DMN3065LW；SOT23候选Qg更高，改为同封装外伸焊盘。; LCSC (none) -> C150506
- Q3: BOM Comments (none) -> 保留原型号/封装；本轮逐项复核，关键动态参数未有充分替代证据。; LCSC (none) -> C82762
- Q6: BOM Comments (none) -> 保留原型号/封装；本轮逐项复核，关键动态参数未有充分替代证据。; LCSC (none) -> C94514
- Q8: BOM Comments (none) -> 保留原型号/封装；本轮逐项复核，关键动态参数未有充分替代证据。; LCSC (none) -> C151010
- R10, R19: footprint Driver:Resistor_SMD__R_0603_1608Metric -> Driver:R_0805_HandSolder; BOM Comments (none) -> 同阻值±1%常用0805；手焊加长焊盘。; LCSC (none) -> C17521; MPN RC0603FR-072R2L -> 0805W8F220KT5E; Manufacturer Yageo -> UNI-ROYAL
- R11, R30: footprint Driver:Resistor_SMD__R_0603_1608Metric -> Driver:R_0805_HandSolder; BOM Comments (none) -> 同阻值±1%常用0805；手焊加长焊盘。; LCSC (none) -> C149504; MPN RC0603FR-07100KL -> 0805W8F1003T5E; Manufacturer Yageo -> UNI-ROYAL
- R12: footprint Driver:Resistor_SMD__R_0603_1608Metric -> Driver:R_0805_HandSolder; BOM Comments (none) -> 同阻值±1%常用0805；手焊加长焊盘。; LCSC (none) -> C4310; MPN RC0603FR-071K5L -> 0805W8F1501T5E; Manufacturer Yageo -> UNI-ROYAL
- R13, R2, R3: footprint Driver:Resistor_SMD__R_0603_1608Metric -> Driver:R_0805_HandSolder; BOM Comments (none) -> 同阻值±1%常用0805；手焊加长焊盘。; LCSC (none) -> C17514; MPN RC0603FR-071ML -> 0805W8F1004T5E; Manufacturer Yageo -> UNI-ROYAL
- R17: value 400k ohm -> 200k ohm; footprint Driver:Resistor_SMD__R_0603_1608Metric -> Driver:R_0805_HandSolder; BOM Comments (none) -> 同阻值±1%常用0805；手焊加长焊盘。; LCSC (none) -> C17539; MPN RC0603FR-07400KL -> 0805W8F2003T5E; Manufacturer Yageo -> UNI-ROYAL
- R18: footprint Driver:Resistor_SMD__R_0603_1608Metric -> Driver:R_0805_HandSolder; BOM Comments (none) -> 同阻值±1%常用0805；手焊加长焊盘。; LCSC (none) -> C17490; MPN RC0603FR-0716KL -> 0805W8F1602T5E; Manufacturer Yageo -> UNI-ROYAL
- R49: BOM Comments (none) -> 保留原型号/封装；本轮逐项复核，关键动态参数未有充分替代证据。; LCSC (none) -> C96345
- R7: footprint Driver:Resistor_SMD__R_0603_1608Metric -> Driver:R_0805_HandSolder; BOM Comments (none) -> 同阻值±1%常用0805；手焊加长焊盘。; LCSC (none) -> C137518; MPN RC0603FR-074K3L -> RC0805FR-074K3L; Manufacturer Yageo -> YAGEO
- R8: footprint Driver:Resistor_SMD__R_0603_1608Metric -> Driver:R_0805_HandSolder; BOM Comments (none) -> 同阻值±1%常用0805；手焊加长焊盘。; LCSC (none) -> C137599; MPN RC0603FR-07110KL -> RC0805FR-07110KL; Manufacturer Yageo -> YAGEO
- U5: BOM Comments (none) -> 保留原型号/封装；本轮逐项复核，关键动态参数未有充分替代证据。; LCSC (none) -> C2681320
Connections:
- net VGL: now also R50.1; no longer R17.1
- new net VGL_FB_MID: R17.1, R50.2

Commit message: feat(pcb): release v0.9 with fee-waived resistor selections
Parts:
- C28: value 2.2uF/50V -> 4.7uF/50V; BOM Comments 保留原型号/封装；本轮逐项复核，关键动态参数未有充分替代证据。 -> v0.8 国内现货降本；详见降本审核-v0.8.md; LCSC (none) -> C86052; MPN GRM32ER71H225KA88L -> GRM32ER71H475KA88L
- C36: BOM Comments 保留原型号/封装；本轮逐项复核，关键动态参数未有充分替代证据。 -> v0.7 嘉立创国内现货替代；参数及实测边界见三组现货替代-v0.7.md; LCSC (none) -> C29925; MPN C0805C102J5GACTU -> 0805CG102J500NT; Manufacturer KEMET -> FH
- D1, D2: LCSC (none) -> C151335
- D3, D5, D6: value BAT54S-7-F -> BAT54SLT1G; BOM Comments 保留原型号/封装；本轮逐项复核，关键动态参数未有充分替代证据。 -> v0.8 国内现货降本；详见降本审核-v0.8.md; LCSC C83574 -> C19726; MPN BAT54S-7-F -> BAT54SLT1G; Manufacturer Diodes -> onsemi
- D4: LCSC (none) -> C124188
- L1, L2, L3: footprint Driver:Inductor_SMD__L_Coilcraft_MSS1246T-XXX -> Driver:L_JIERR_PCR1040; BOM Comments 保留原型号/封装；本轮逐项复核，关键动态参数未有充分替代证据。 -> v0.7 嘉立创国内现货替代；参数及实测边界见三组现货替代-v0.7.md; LCSC (none) -> C53896892; MPN MSS1246-153MLC -> PCR1040-150-M; Manufacturer Coilcraft -> JIERR
- Q7: LCSC (none) -> C6628419
- R10, R19: AssemblyMethod (none) -> SMT; BOM Comments 同阻值±1%常用0805；手焊加长焊盘。 -> v0.9 三组电阻免换料费；详见三组电阻免换料费改版-v0.9.md; ExceptionDecision (none) -> 2026-10-10 user authorized three resistor groups only; all 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; FeeEvidence (none) -> https://www.jlc-smt.com/lcsc/search?q=C17521 | 基础库 (免换料费); LibraryCategory (none) -> 基础库; StockQueriedAt (none) -> 2026-10-10T13:26:26.075Z
- R17: AssemblyMethod (none) -> SMT; BOM Comments 同阻值±1%常用0805；手焊加长焊盘。 -> v0.9 三组电阻免换料费；详见三组电阻免换料费改版-v0.9.md; ExceptionDecision (none) -> 2026-10-10 user authorized three resistor groups only; all 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; FeeEvidence (none) -> https://www.jlc-smt.com/lcsc/search?q=C17539 | 基础库 (免换料费); LibraryCategory (none) -> 基础库; StockQueriedAt (none) -> 2026-10-10T13:26:27.744Z
- R18: BOM Comments 同阻值±1%常用0805；手焊加长焊盘。 -> v0.8 国内现货降本；详见降本审核-v0.8.md; LCSC C17490 -> C2774511; MPN 0805W8F1602T5E -> HP05W3F1602T5E
- R49: BOM Comments 保留原型号/封装；本轮逐项复核，关键动态参数未有充分替代证据。 -> v0.8 国内现货降本；详见降本审核-v0.8.md; LCSC C96345 -> C17477; MPN RC0805JR-070RL -> 0805W8F0000T5E; Manufacturer Yageo -> UNI-ROYAL
- R50: AssemblyMethod (none) -> SMT; BOM Comments 与R17串联：200k+200k=400k，±1%最坏误差，±100ppm/℃。 -> v0.9 三组电阻免换料费；详见三组电阻免换料费改版-v0.9.md; ExceptionDecision (none) -> 2026-10-10 user authorized three resistor groups only; all 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; FeeEvidence (none) -> https://www.jlc-smt.com/lcsc/search?q=C17539 | 基础库 (免换料费); LibraryCategory (none) -> 基础库; StockQueriedAt (none) -> 2026-10-10T13:26:27.744Z
- R7: AssemblyMethod (none) -> SMT; BOM Comments 同阻值±1%常用0805；手焊加长焊盘。 -> v0.9 三组电阻免换料费；详见三组电阻免换料费改版-v0.9.md; ExceptionDecision (none) -> 2026-10-10 user authorized three resistor groups only; all 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; FeeEvidence (none) -> https://www.jlc-smt.com/lcsc/search?q=C17667 | 扩展库 (免换料费); LCSC C137518 -> C17667; LibraryCategory (none) -> SMT优选合作（扩展库免换料费）; MPN RC0805FR-074K3L -> 0805W8F4301T5E; Manufacturer YAGEO -> UNI-ROYAL; StockQueriedAt (none) -> 2026-10-10T13:18:09.034Z
- R8: BOM Comments 同阻值±1%常用0805；手焊加长焊盘。 -> v0.8 国内现货降本；详见降本审核-v0.8.md; LCSC C137599 -> C5140228; MPN RC0805FR-07110KL -> SCR0805F110K; Manufacturer YAGEO -> VO
- U1, U2, U3: LCSC (none) -> C2073442

Commit message: hardware: use Murata C440198 0805 capacitors and release v0.10
Parts:
- C13, C15, C20: value 10uF/50V -> 10uF/50V X5R; footprint Driver:Capacitor_SMD__C_1210_3225Metric -> Driver:C_0805_HandSolder; AssemblyMethod (none) -> SMT; BOM Comments 保留原型号/封装；本轮逐项复核，关键动态参数未有充分替代证据。 -> v0.10 E01指定C440198；X5R/0805；偏压容量与纹波等效未验证；详见E01改版-v0.10.md; ExceptionDecision (none) -> 2026-10-11 user explicitly selected C440198 for E01; protot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; FeeEvidence (none) -> https://item.szlcsc.com/439567.html | SMT基础库; LCSC C77102 -> C440198; LibraryCategory (none) -> 基础库; MPN GRM32ER71H106KA12L -> GRM21BR61H106KE43L; StockQueriedAt (none) -> 2026-10-11T11:28:17.670114+08:00

Commit message: feat(pcb): adopt 17 basic-library groups and release v0.11 prototype
Parts:
- C12, C14, C16, C19, C21, C29, C30: footprint Driver:Capacitor_SMD__C_1210_3225Metric -> Driver:C_1206_HandSolder; AssemblyMethod (none) -> SMT; BOM Comments 保留原型号/封装；本轮逐项复核，关键动态参数未有充分替代证据。 -> 2026-10-11 user selected 3+14 groups; E05; PROTOTYPE ONLY -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; ExceptionDecision (none) -> 2026-10-11 user selected 3+14 groups; E05; PROTOTYPE ONLY -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; FeeEvidence (none) -> https://item.szlcsc.com/30577.html | SMT基础库; LCSC C86052 -> C29823; LibraryCategory (none) -> 基础库; MPN GRM32ER71H475KA88L -> 1206B475K500NT; Manufacturer Murata -> FH; StockQueriedAt (none) -> 2026-10-11T14:08:16.690356+08:00
- C17, C23, C24: footprint Driver:Capacitor_SMD__C_0805_2012Metric -> Driver:C_0805_HandSolder; AssemblyMethod (none) -> SMT; BOM Comments 保留原型号/封装；本轮逐项复核，关键动态参数未有充分替代证据。 -> 2026-10-11 user selected 3+14 groups; E13; PROTOTYPE ONLY -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; ExceptionDecision (none) -> 2026-10-11 user selected 3+14 groups; E13; PROTOTYPE ONLY -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; FeeEvidence (none) -> https://item.szlcsc.com/14623.html | SMT基础库; LCSC C86043 -> C13967; LibraryCategory (none) -> 基础库; MPN GRM21BR71H474KA88L -> CL21B474KBFNNNE; Manufacturer Murata -> Samsung Electro-Mechanics; StockQueriedAt (none) -> 2026-10-11T14:08:21.232417+08:00
- C18: value 220nF/50V -> 100nF/100V; footprint Driver:Capacitor_SMD__C_0805_2012Metric -> Driver:C_0805_HandSolder; AssemblyMethod (none) -> SMT; BOM Comments 保留原型号/封装；本轮逐项复核，关键动态参数未有充分替代证据。 -> 2026-10-11 user selected 3+14 groups; E18; PROTOTYPE ONLY -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; ExceptionDecision (none) -> 2026-10-11 user selected 3+14 groups; E18; PROTOTYPE ONLY -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; FeeEvidence (none) -> https://item.szlcsc.com/28983.html | SMT基础库; LCSC C86042 -> C28233; LibraryCategory (none) -> 基础库; MPN GRM21BR71H224KA01L -> CL21B104KCFNNNE; Manufacturer Murata -> Samsung Electro-Mechanics; StockQueriedAt (none) -> 2026-10-11T14:08:23.039107+08:00
- C22, C25: footprint Driver:Capacitor_SMD__C_0805_2012Metric -> Driver:C_0805_HandSolder; AssemblyMethod (none) -> SMT; BOM Comments 保留原型号/封装；本轮逐项复核，关键动态参数未有充分替代证据。 -> 2026-10-11 user selected 3+14 groups; E19; PROTOTYPE ONLY -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; ExceptionDecision (none) -> 2026-10-11 user selected 3+14 groups; E19; PROTOTYPE ONLY -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; FeeEvidence (none) -> https://item.szlcsc.com/29074.html | SMT基础库; LCSC C77083 -> C28323; LibraryCategory (none) -> 基础库; MPN GRM21BR71H105KA12L -> CL21B105KBFNNNE; Manufacturer Murata -> Samsung Electro-Mechanics; StockQueriedAt (none) -> 2026-10-11T14:08:23.138241+08:00
- C26: footprint Driver:C_0805_HandSolder -> Driver:Capacitor_SMD__C_0603_1608Metric; AssemblyMethod (none) -> SMT; BOM Comments 47nF/50V X7R±10%；风华0805，保留耐压，动态波形待实测。 -> 2026-10-11 user selected 3+14 groups; E12; PROTOTYPE ONLY -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; ExceptionDecision (none) -> 2026-10-11 user selected 3+14 groups; E12; PROTOTYPE ONLY -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; FeeEvidence (none) -> https://item.szlcsc.com/1974.html | SMT基础库; LCSC C1745 -> C1622; LibraryCategory (none) -> 基础库; MPN 0805B473K500NT -> CL10B473KB8NNNC; Manufacturer FH -> Samsung Electro-Mechanics; StockQueriedAt (none) -> 2026-10-11T14:08:26.139847+08:00
- C28: footprint Driver:Capacitor_SMD__C_1210_3225Metric -> Driver:C_1206_HandSolder; AssemblyMethod (none) -> SMT; BOM Comments v0.8 国内现货降本；详见降本审核-v0.8.md -> 2026-10-11 user selected 3+14 groups; E05; PROTOTYPE ONLY -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; ExceptionDecision (none) -> 2026-10-11 user selected 3+14 groups; E05; PROTOTYPE ONLY -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; FeeEvidence (none) -> https://item.szlcsc.com/30577.html | SMT基础库; LCSC C86052 -> C29823; LibraryCategory (none) -> 基础库; MPN GRM32ER71H475KA88L -> 1206B475K500NT; Manufacturer Murata -> FH; StockQueriedAt (none) -> 2026-10-11T14:08:16.690356+08:00
- C31, C32: footprint Driver:Capacitor_SMD__C_1210_3225Metric -> Driver:C_1206_HandSolder; AssemblyMethod (none) -> SMT; BOM Comments 保留原型号/封装；本轮逐项复核，关键动态参数未有充分替代证据。 -> 2026-10-11 user selected 3+14 groups; E04; PROTOTYPE ONLY -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; ExceptionDecision (none) -> 2026-10-11 user selected 3+14 groups; E04; PROTOTYPE ONLY -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; FeeEvidence (none) -> https://item.szlcsc.com/15681.html | SMT基础库; LCSC C88154 -> C15008; LibraryCategory (none) -> 基础库; MPN GRM32ER60J107ME20L -> CL31A107MQHNNNE; Manufacturer Murata -> Samsung Electro-Mechanics; StockQueriedAt (none) -> 2026-10-11T14:12:33.174140+08:00
- C33: value 100nF/50V -> 100nF/100V; AssemblyMethod (none) -> SMT; BOM Comments 100nF/50V X7R±10%；0603增大为0805。 -> 2026-10-11 user selected 3+14 groups; E21; parametric revie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; ExceptionDecision (none) -> 2026-10-11 user selected 3+14 groups; E21; parametric revie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; FeeEvidence (none) -> https://item.szlcsc.com/28983.html | SMT基础库; LCSC C1711 -> C28233; LibraryCategory (none) -> 基础库; MPN CL21B104KBCNNNC -> CL21B104KCFNNNE; Manufacturer Samsung -> Samsung Electro-Mechanics; StockQueriedAt (none) -> 2026-10-11T14:08:23.039107+08:00
- C36: value 1nF/50V C0G -> 100pF/50V C0G; footprint Driver:Capacitor_SMD__C_0805_2012Metric -> Driver:Capacitor_SMD__C_0603_1608Metric; AssemblyMethod (none) -> SMT; BOM Comments v0.7 嘉立创国内现货替代；参数及实测边界见三组现货替代-v0.7.md -> 2026-10-11 user selected 3+14 groups; E14; PROTOTYPE ONLY -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; ExceptionDecision (none) -> 2026-10-11 user selected 3+14 groups; E14; PROTOTYPE ONLY -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; FeeEvidence (none) -> https://item.szlcsc.com/15530.html | SMT基础库; LCSC C29925 -> C14858; LibraryCategory (none) -> 基础库; MPN 0805CG102J500NT -> CL10C101JB8NNNC; Manufacturer FH -> Samsung Electro-Mechanics; StockQueriedAt (none) -> 2026-10-11T14:16:46.940464+08:00
- D1, D2: value MBR230S1F-7 -> SS34; footprint Driver:Diode_SMD__D_SOD-123F -> Driver:D_SMA_HandSolder; AssemblyMethod (none) -> SMT; BOM Comments 保留原型号/封装；本轮逐项复核，关键动态参数未有充分替代证据。 -> 2026-10-11 user selected 3+14 groups; E11; PROTOTYPE ONLY -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; ExceptionDecision (none) -> 2026-10-11 user selected 3+14 groups; E11; PROTOTYPE ONLY -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; FeeEvidence (none) -> https://item.szlcsc.com/9178.html | SMT基础库; LCSC C151335 -> C8678; LibraryCategory (none) -> 基础库; MPN MBR230S1F-7 -> SS34; Manufacturer Diodes -> MDD(Microdiode Semiconductor); StockQueriedAt (none) -> 2026-10-11T14:12:14.414733+08:00
- D4: value B0530W-7-F -> B5819W SL; AssemblyMethod (none) -> SMT; BOM Comments 保留原型号/封装；本轮逐项复核，关键动态参数未有充分替代证据。 -> 2026-10-11 user selected 3+14 groups; E17; PROTOTYPE ONLY -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; ExceptionDecision (none) -> 2026-10-11 user selected 3+14 groups; E17; PROTOTYPE ONLY -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; FeeEvidence (none) -> https://item.szlcsc.com/9093.html | SMT基础库; LCSC C124188 -> C8598; LibraryCategory (none) -> 基础库; MPN B0530W-7-F -> B5819W SL; Manufacturer Diodes -> JSCJ; StockQueriedAt (none) -> 2026-10-11T14:08:46.105804+08:00
- Q1, Q4: value DMN3065LW-7 -> AO3400A; footprint Driver:SOT323_HandSolder -> Driver:Package_TO_SOT_SMD__SOT-23; AssemblyMethod (none) -> SMT; BOM Comments 保留DMN3065LW；SOT23候选Qg更高，改为同封装外伸焊盘。 -> 2026-10-11 user selected 3+14 groups; E09; PROTOTYPE ONLY -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; ExceptionDecision (none) -> 2026-10-11 user selected 3+14 groups; E09; PROTOTYPE ONLY -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; FeeEvidence (none) -> https://item.szlcsc.com/21629.html | SMT基础库; LCSC C150506 -> C20917; LibraryCategory (none) -> 基础库; MPN DMN3065LW-7 -> AO3400A; Manufacturer Diodes -> AOS; StockQueriedAt (none) -> 2026-10-11T14:08:47.487158+08:00
- Q6: value MMBT3904-7-F -> MMBT3904; AssemblyMethod (none) -> SMT; BOM Comments 保留原型号/封装；本轮逐项复核，关键动态参数未有充分替代证据。 -> 2026-10-11 user selected 3+14 groups; E15; PROTOTYPE ONLY -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; ExceptionDecision (none) -> 2026-10-11 user selected 3+14 groups; E15; PROTOTYPE ONLY -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; FeeEvidence (none) -> https://item.szlcsc.com/21237.html | SMT基础库; LCSC C94514 -> C20526; LibraryCategory (none) -> 基础库; MPN MMBT3904-7-F -> MMBT3904(RANGE:100-300); Manufacturer Diodes -> JSCJ; StockQueriedAt (none) -> 2026-10-11T14:08:38.028013+08:00
- Q7: value PJA3433_R1_00001 -> AO3401A; AssemblyMethod (none) -> SMT; BOM Comments 保留原型号/封装；本轮逐项复核，关键动态参数未有充分替代证据。 -> 2026-10-11 user selected 3+14 groups; E08; PROTOTYPE ONLY -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; ExceptionDecision (none) -> 2026-10-11 user selected 3+14 groups; E08; PROTOTYPE ONLY -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; FeeEvidence (none) -> https://item.szlcsc.com/15801.html | SMT基础库; LCSC C6628419 -> C15127; LibraryCategory (none) -> 基础库; MPN PJA3433_R1_00001 -> AO3401A; Manufacturer Panjit -> AOS; StockQueriedAt (none) -> 2026-10-11T14:08:47.923870+08:00
- Q8: value DMP3068L-7 -> AO3401A; AssemblyMethod (none) -> SMT; BOM Comments 保留原型号/封装；本轮逐项复核，关键动态参数未有充分替代证据。 -> 2026-10-11 user selected 3+14 groups; E10; PROTOTYPE ONLY -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; ExceptionDecision (none) -> 2026-10-11 user selected 3+14 groups; E10; PROTOTYPE ONLY -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; FeeEvidence (none) -> https://item.szlcsc.com/15801.html | SMT基础库; LCSC C151010 -> C15127; LibraryCategory (none) -> 基础库; MPN DMP3068L-7 -> AO3401A; Manufacturer Diodes -> AOS; StockQueriedAt (none) -> 2026-10-11T14:08:47.923870+08:00
- R18: value 16k ohm -> 15k ohm; AssemblyMethod (none) -> SMT; BOM Comments v0.8 国内现货降本；详见降本审核-v0.8.md -> 2026-10-11 user selected 3+14 groups; E20; parametric revie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; ExceptionDecision (none) -> 2026-10-11 user selected 3+14 groups; E20; parametric revie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; FeeEvidence (none) -> https://item.szlcsc.com/18163.html | SMT基础库; LCSC C2774511 -> C17475; LibraryCategory (none) -> 基础库; MPN HP05W3F1602T5E -> 0805W8F1502T5E; StockQueriedAt (none) -> 2026-10-11T14:16:44.474570+08:00
- R8: value 110k ohm -> 100k ohm; AssemblyMethod (none) -> SMT; BOM Comments v0.8 国内现货降本；详见降本审核-v0.8.md -> 2026-10-11 user selected 3+14 groups; E22; parametric revie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; ExceptionDecision (none) -> 2026-10-11 user selected 3+14 groups; E22; parametric revie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; FeeEvidence (none) -> https://item.szlcsc.com/160838.html | SMT基础库; LCSC C5140228 -> C149504; LibraryCategory (none) -> 基础库; MPN SCR0805F110K -> 0805W8F1003T5E; Manufacturer VO -> UNI-ROYAL; StockQueriedAt (none) -> 2026-10-11T14:16:45.969921+08:00
Connections:
- net REG_VGN: no longer R18.2
- net VGH: no longer R8.2
- new net R18_FB_MID: R18.2
- new net R8_FB_MID: R8.2
